File: StepperServo.kicad_pcb (KiCad board)
At the start: 2 copper layers, 35.5 x 35.5 mm, 90 parts, among them J1 Conn_01x01_Female, J2 Conn_01x01_Female, J3 Conn_01x04_Male, J4 I2C_External, J6 Conn_TempMotor, SW1 SW_MainOffset, SW2 SW_LeftWheelOffset, SW4 SW_Reset, U1 TC1185, U2 SN65HVD232, U3 TMC2209-LA, U4 24LC64, U5 STM32F103RETx, U6 AS5600, U7 INA180A1, Y1 ABM3B-16MHz

Commit message: wip layout
Parts:
- C17, C18, C19, C20, C21, C22, C36, C37, R20: moved to B.Cu
- R1: value R -> 1.1R
- moved C8 100.6 mm to (77.8, 121.2)
- moved C15 99.7 mm to (83.2, 116.1)
- moved R5 94.5 mm to (80.0, 129.4)
- moved R6 90.5 mm to (112.4, 137.5)
- moved C11 88.0 mm to (99.1, 118.6)
- moved C37 85.0 mm to (133.1, 116.1)
- moved C32 85.0 mm to (127.9, 114.6)
- moved R20 83.7 mm to (132.9, 114.2)
- moved C13 83.2 mm to (99.0, 125.7)
- moved R8 83.2 mm to (102.9, 135.7)
- moved R18 80.6 mm to (127.5, 111.5)
- moved C1 80.5 mm to (153.0, 125.6)
- moved TH1 80.2 mm to (127.5, 113.1)
- moved R2 78.7 mm to (157.0, 125.9)
- moved C12 78.1 mm to (88.8, 121.5)
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Connections:
- C17 pad 1: /StepperDriver/coilB_2 -> /StepperDriver/coilA_2
- C19 pad 1: /StepperDriver/coilB_1 -> /StepperDriver/coilA_1
- C20 pad 1: /StepperDriver/coilA_1 -> /StepperDriver/coilB_1
- C22 pad 1: /StepperDriver/coilA_2 -> /StepperDriver/coilB_2
- C38 pad 2: GNDD -> GND
- C39 pad 2: GNDD -> GND
- J3 pad 1: /StepperDriver/coilB_2 -> /StepperDriver/coilA_2
- J3 pad 2: /StepperDriver/coilB_1 -> /StepperDriver/coilA_1
- J3 pad 3: /StepperDriver/coilA_1 -> /StepperDriver/coilB_1
- J3 pad 4: /StepperDriver/coilA_2 -> /StepperDriver/coilB_2
- U6 pad 4: GNDD -> GND
- U6 pad 5: GNDD -> GND
- U6 pad 8: GNDD -> GND
Other:
- copper layers 2 -> 4

Commit message: wip layout
Parts:
- C10, C11, C12, C13, C14, C15: moved to B.Cu
- moved C15 66.1 mm to (147.2, 99.6), turned to 180 degrees
- moved C12 65.8 mm to (151.1, 100.2)
- moved C10 53.3 mm to (144.9, 96.5)
- moved C13 52.7 mm to (144.1, 98.4)
- moved C14 46.5 mm to (144.2, 109.5)
- moved C11 44.9 mm to (143.4, 111.4)
- moved C18 15.5 mm to (141.2, 109.5), turned to 180 degrees
- moved OPT1 10.2 mm to (157.6, 94.8), turned to 247 degrees
- moved C21 9.96 mm to (141.1, 98.6), turned to 180 degrees
- moved R3 8.10 mm to (97.9, 119.9)
- moved C9 7.80 mm to (97.9, 117.9)
- moved R9 4.35 mm to (141.2, 106.8), turned to 0 degrees
- moved U3 2.24 mm to (145.8, 104.1)
- moved R10 1.98 mm to (141.2, 101.3), turned to 0 degrees
- moved C22 1.43 mm to (135.7, 99.2), turned to 270 degrees
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Connections:
- U5 pad 58: (no net) -> /MCU/I2C1_SCL
- U5 pad 59: (no net) -> /MCU/I2C1_SDA
Routing:
- net GND: track 0.00 -> 24.6 mm, vias 0 -> 10
- net /StepperDriver/~EN: track 0.00 -> 5.98 mm
- net /StepperDriver/chargePumpIn: track 0.00 -> 2.88 mm
- net /StepperDriver/coilA_2: track 0.00 -> 2.81 mm, vias 0 -> 2
- net /StepperDriver/coilB_2: track 0.00 -> 2.79 mm, vias 0 -> 2
- net /StepperDriver/senseCoilA: track 0.00 -> 2.74 mm
- net /StepperDriver/senseCoilB: track 0.00 -> 2.70 mm
- net /StepperDriver/chargePumpOut: track 0.00 -> 2.30 mm
- net /StepperDriver/coilB_1: track 0.00 -> 2.25 mm, vias 0 -> 2
- net /StepperDriver/coilA_1: track 0.00 -> 2.19 mm, vias 0 -> 2
- net /StepperDriver/chargePumpVoltage: track 0.00 -> 1.98 mm
- net VCC: track 0.00 -> 0.07 mm, vias 0 -> 4
- added copper zone on B.Cu, net /StepperDriver/coilA_1
- added copper zone on In1.Cu, net /StepperDriver/coilA_1
- added copper zone on B.Cu, net /StepperDriver/coilA_2
- added copper zone on In1.Cu, net /StepperDriver/coilA_2
- added copper zone on B.Cu, net /StepperDriver/coilB_1
- added copper zone on In1.Cu, net /StepperDriver/coilB_1
- added copper zone on B.Cu, net /StepperDriver/coilB_2
- added copper zone on In1.Cu, net /StepperDriver/coilB_2
- added copper zone on B.Cu, net /StepperDriver/senseCoilA
- added copper zone on B.Cu, net /StepperDriver/senseCoilB
- added copper zone on B.Cu, net GND
- added copper zone on In2.Cu, net GND
- added copper zone on B.Cu, net VCC
- added copper zone on In1.Cu, net VCC
Other:
- net class Default: clearance 0.2 -> 0.254; via_dia 0.8 -> 0.6; via_drill 0.4 -> 0.3
- net class smol added: clearance 0.254, trace_width 0.17, via_dia 0.6, via_drill 0.3
- rule trace_clearance: 0.2 -> 0.254
- rule trace_min: 0.2 -> 0.15

Commit message: wip layout
Parts:
- removed C29, C31, C32, C36, C37: 100nF 35V, Capacitor_SMD:C_0603_1608Metric
- removed C38: 10uF 35V, Capacitor_SMD:C_1206_3216Metric
- removed D2: LED, LED_SMD:LED_0603_1608Metric
- removed R18: 10k, Resistor_SMD:R_0603_1608Metric
- removed R8: 220, Resistor_SMD:R_0603_1608Metric
- removed SW1: SW_MainOffset, standardContent:SW_SPST_PTS636_SM25F
- removed SW2: SW_LeftWheelOffset, standardContent:SW_SPST_PTS636_SM25F
- removed TH1: 10k @ 25°C, Resistor_SMD:R_0603_1608Metric
- removed U4: 24LC64, Package_TO_SOT_SMD:SOT-23-5
- C16, C8, R11, R7, SW4: moved to B.Cu
- moved C8 72.3 mm to (149.0, 108.7), turned to 270 degrees
- moved C16 67.9 mm to (150.4, 101.0)
- moved R4 67.9 mm to (173.1, 105.5)
- moved R6 67.9 mm to (173.1, 107.1)
- moved SW4 64.2 mm to (147.1, 91.0), turned to 0 degrees
- moved R11 60.6 mm to (147.3, 109.0), turned to 270 degrees
- moved R7 59.2 mm to (147.8, 111.9)
- moved R5 57.2 mm to (128.6, 99.2)
- moved R3 51.8 mm to (149.4, 114.5), turned to 270 degrees
- moved R23 51.4 mm to (179.1, 112.9)
- moved C40 50.8 mm to (179.1, 111.4)
- moved C7 50.8 mm to (175.6, 111.6)
- moved C9 49.9 mm to (147.7, 114.6), turned to 270 degrees
- moved C25 46.9 mm to (157.5, 104.7)
- moved C35 46.1 mm to (163.2, 104.7), turned to 270 degrees
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Connections:
- OPT1 pad 4: (no net) -> /MCU/endstopRight
- R21 pad 1: (no net) -> /MCU/LED_RED
- R22 pad 1: (no net) -> /MCU/LED_GREEN
- U3 pad 10: +3V3 -> GND
- U3 pad 11: /StepperDriver/Diag -> (no net)
- U3 pad 16: (no net) -> /StepperDriver/Step
- U3 pad 19: (no net) -> /StepperDriver/Direction
- U3 pad 9: +3V3 -> GND
- U5 pad 15: (no net) -> /MCU/LED_GREEN
- U5 pad 16: (no net) -> /MCU/LED_RED
- U5 pad 2: (no net) -> /MCU/endstopRight
- U5 pad 29: (no net) -> /MCU/I2C2_SCL
- U5 pad 30: (no net) -> /MCU/I2C2_SDA
- U5 pad 50: (no net) -> /StepperDriver/Step
- U5 pad 51: (no net) -> /StepperDriver/Direction
Routing:
- net GND: track 24.6 -> 131.7 mm, vias 10 -> 34
- net +3V3: track 0.00 -> 101.9 mm, vias 0 -> 11
- net /MCU/~RST: track 0.00 -> 47.2 mm, vias 0 -> 4
- net +5V: track 0.00 -> 35.2 mm, vias 0 -> 1
- net /MCU/I2C2_SDA: track 0.00 -> 33.2 mm, vias 0 -> 1
- net /MCU/I2C2_SCL: track 0.00 -> 26.0 mm, vias 0 -> 1
- net Net-(J_CAN1-Pad2): track 0.00 -> 22.3 mm, vias 0 -> 1
- net /StepperDriver/Direction: track 0.00 -> 22.1 mm
- net /MCU/tempMotor: track 0.00 -> 18.0 mm
- net /MCU/I2C1_SDA: track 0.00 -> 16.8 mm, vias 0 -> 1
- net Net-(R23-Pad2): track 0.00 -> 16.6 mm
- net /StepperDriver/Step: track 0.00 -> 14.7 mm
- net Net-(J_CAN1-Pad1): track 0.00 -> 14.0 mm, vias 0 -> 1
- net VCC: track 0.07 -> 13.9 mm, vias 4 -> 7
- net /MCU/SWO: track 0.00 -> 12.5 mm, vias 0 -> 1
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- added copper zone on B.Cu, net +3V3
- added copper zone on F.Cu, net GND
- added copper zone on In1.Cu, net GND
- added copper zone on F.Cu, net Net-(J1-Pad1)
- added copper zone on F.Cu, net VCC

Commit message: Finished v1 layout Added pictures to readme
Parts:
- R16, R5: moved to B.Cu
- moved R23 28.0 mm to (151.1, 113.9), turned to 270 degrees
- moved R5 22.0 mm to (150.4, 96.1), turned to 180 degrees
- moved C40 18.7 mm to (160.6, 108.9), turned to 270 degrees
- moved R6 17.4 mm to (155.8, 109.0), turned to 90 degrees
- moved R4 16.2 mm to (157.3, 109.0), turned to 90 degrees
- moved C7 13.7 mm to (162.1, 108.9), turned to 270 degrees
- moved R16 1.53 mm to (154.8, 90.8), turned to 0 degrees
- moved C25 0.20 mm to (157.7, 104.7)
- moved C16 0.10 mm to (150.4, 101.1)
- turned R14 to 90 degrees
- turned R15 to 90 degrees
Connections:
- R4 pad 2: (no net) -> /MCU/Stepper_UART
- U3 pad 11: (no net) -> /StepperDriver/Diag
- U5 pad 23: (no net) -> /inputCurrent
- U5 pad 24: (no net) -> /MCU/tempMotor
- U5 pad 3: (no net) -> /StepperDriver/Diag
- U5 pad 4: (no net) -> /StepperDriver/~EN
- U5 pad 53: (no net) -> /MCU/Stepper_UART
Routing:
- net +5V: track 35.2 -> 85.7 mm, vias 1 -> 2
- net +3V3: track 101.9 -> 138.7 mm, vias 11 -> 12
- net /MCU/tempMotor: track 18.0 -> 53.2 mm, vias 0 -> 5
- net /inputCurrent: track 0.00 -> 23.8 mm, vias 0 -> 3
- net /StepperDriver/~EN: track 5.98 -> 26.5 mm, vias 0 -> 3
- net /StepperDriver/Diag: track 0.00 -> 15.1 mm
- net Net-(R23-Pad2): track 16.6 -> 29.2 mm, vias 0 -> 2
- net GND: track 131.7 -> 143.2 mm, vias 34 -> 40
- net /MCU/Stepper_UART: track 0.00 -> 7.83 mm, vias 0 -> 1
- net Net-(J_CAN1-Pad2): track 22.3 -> 14.8 mm
- net Net-(R4-Pad1): track 3.96 -> 11.4 mm, vias 0 -> 1
- net /MCU/I2C1_SDA: track 16.8 -> 13.5 mm
- net Net-(OPT1-Pad1): track 3.64 -> 2.31 mm, vias 1 -> 0
- net (no net): track 0.95 -> 0.00 mm
- net /CAN_TX: track 8.00 -> 7.28 mm
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Other:
- net class Default: clearance 0.254 -> 0.15
- net class smol: clearance 0.254 -> 0.15
- rule trace_clearance: 0.254 -> 0.15
- board text added: "2021"
- board text added: "A1"
- board text added: "A2"
- board text added: "Albrecht"
- board text added: "B1"
- board text added: "B2"
- board text added: "CAN"
- board text added: "ExtSen"
- board text added: "Gnd"
- board text added: "SWD"
- board text added: "Stepper Servo v1"
- board text added: "Tmp"
- board text added: "Vcc"

Commit message: exported step file exported production files fixed omron photo interruper 3d model
Parts:
- R1: value 1.1R -> 0.11
